File: eagle/hh.brd (EAGLE design)
At the start: 169.7 x 51.9 mm, 0 parts

Commit message: updates to eagle files
Parts:
- added R1, R2, R3, R4, R5, R6: 4.7K, rcl:0207/5V
- added S1, S2, S3, S4: (no value), switch-omron:B3F-10XX
- added U$1: ESP12E_DEVKIT, ESP12E_DEVKIT:ESP12E_DEVKIT
Changed lines of the file:
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@@
 <layer number="51" name="tDocu" color="7" fill="1" visible="yes" active="yes"/>
 <layer number="52" name="bDocu" color="7" fill="1" visible="yes" active="yes"/>
+<layer number="90" name="Modules" color="5" fill="1" visible="no" active="no"/>
+<layer number="91" name="Nets" color="2" fill="1" visible="no" active="no"/>
+<layer number="92" name="Busses" color="1" fill="1" visible="no" active="no"/>
+<layer number="93" name="Pins" color="2" fill="1" visible="no" active="no"/>
+<layer number="94" name="Symbols" color="4" fill="1" visible="no" active="no"/>
+<layer number="95" name="Names" color="7" fill="1" visible="no" active="no"/>
+<layer number="96" name="Values" color="7" fill="1" visible="no" active="no"/>
+<layer number="97" name="Info" color="7" fill="1" visible="no" active="no"/>
+<layer number="98" name="Guide" color="6" fill="1" visible="no" active="no"/>
 </layers>
 <board>
@@
 </autorouter>
 <elements>
+<element name="S1" library="switch-omron" package="B3F-10XX" value="" x="8.89" y="41.91" rot="R270">
+<attribute name="OC_NEWARK" value="36M3542" x="8.89" y="41.91" size="1.778" layer="27" rot="R270" display="off"/>
+<attribute name="MPN" value="B3F-1000" x="8.89" y="41.91" size="1.778" layer="27" rot="R270" display="off"/>
+<attribute name="MF" value="" x="8.89" y="41.91" size="1.778" layer="27" rot="R270" display="off"/>
+<attribute name="OC_FARNELL" value="176432" x="8.89" y="41.91" size="1.778" layer="27" rot="R270" display="off"/>
+</element>
+<element name="S2" library="switch-omron" package="B3F-10XX" value="" x="24.13" y="41.91" rot="R90">
+<attribute name="OC_NEWARK" value="36M3542" x="24.13" y="41.91" size="1.778" layer="27" rot="R90" display="off"/>
+<attribute name="MPN" value="B3F-1000" x="24.13" y="41.91" size="1.778" layer="27" rot="R90" display="off"/>
+<attribute name="MF" value="" x="24.13" y="41.91" size="1.778" layer="27" rot="R90" display="off"/>
+<attribute name="OC_FARNELL" value="176432" x="24.13" y="41.91" size="1.778" layer="27" rot="R90" display="off"/>
+</element>
+<element name="S3" library="switch-omron" package="B3F-10XX" value="" x="36.83" y="41.91" rot="R270">
+<attribute name="OC_NEWARK" value="36M3542" x="36.83" y="41.91" size="1.778" layer="27" rot="R270" display="off"/>
+<attribute name="MPN" value="B3F-1000" x="36.83" y="41.91" size="1.778" layer="27" rot="R270" display="off"/>
+<attribute name="MF" value="" x="36.83" y="41.91" size="1.778" layer="27" rot="R270" display="off"/>
+<attribute name="OC_FARNELL" value="176432" x="36.83" y="41.91" size="1.778" layer="27" rot="R270" display="off"/>
+</element>
+<element name="S4" library="switch-omron" package="B3F-10XX" value="" x="49.53" y="41.91" rot="R270">
+<attribute name="OC_NEWARK" value="36M3542" x="49.53" y="41.91" size="1.778" layer="27" rot="R270" display="off"/>
+<attribute name="MPN" value="B3F-1000" x="49.53" y="41.91" size="1.778" layer="27" rot="R270" display="off"/>
+<attribute name="MF" value="" x="49.53" y="41.91" size="1.778" layer="27" rot="R270" display="off"/>
+<attribute name="OC_FARNELL" value="176432" x="49.53" y="41.91" size="1.778" layer="27" rot="R270" display="off"/>
+</element>
+<element name="U$1" library="ESP12E_DEVKIT" package="ESP12E_DEVKIT" value="ESP12E_DEVKIT" x="68.58" y="26.67" rot="R180"/>
+<element name="R1" library="rcl" package="0207/5V" value="4.7K" x="44.45" y="31.75"/>
+<element name="R2" library="rcl" package="0207/5V" value="4.7K" x="44.45" y="25.4"/>
+<element name="R3" library="rcl" package="0207/5V" value="4.7K" x="44.45" y="20.32"/>
+<element name="R4" library="rcl" package="0207/5V" value="4.7K" x="44.45" y="15.24"/>
+<element name="R5" library="rcl" package="0207/5V" value="4.7K" x="44.45" y="10.16"/>
+<element name="R6" library="rcl" package="0207/5V" value="4.7K" x="44.45" y="5.08"/>
 </elements>
 <signals>

Commit message: design updates
Parts:
- removed R1, R2, R3, R4, R5, R6: 4.7K, rcl:0207/5V
- added H1: MOUNT-HOLE3.2, holes:3,2
- added JP1: OLED, pinhead:1X04
- moved S4 4.58 mm to (45.7, 44.5)
- moved S1 3.59 mm to (11.4, 44.5)
- moved S3 3.59 mm to (34.3, 44.5)
- moved S2 2.84 mm to (22.9, 44.5), turned to 270 degrees
Changed lines of the file:
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@@
 </autorouter>
 <elements>
-<element name="S1" library="switch-omron" package="B3F-10XX" value="" x="8.89" y="41.91" rot="R270">
-<attribute name="OC_NEWARK" value="36M3542" x="8.89" y="41.91" size="1.778" layer="27" rot="R270" display="off"/>
-<attribute name="MPN" value="B3F-1000" x="8.89" y="41.91" size="1.778" layer="27" rot="R270" display="off"/>
-<attribute name="MF" value="" x="8.89" y="41.91" size="1.778" layer="27" rot="R270" display="off"/>
-<attribute name="OC_FARNELL" value="176432" x="8.89" y="41.91" size="1.778" layer="27" rot="R270" display="off"/>
+<element name="S1" library="switch-omron" package="B3F-10XX" value="" x="11.43" y="44.45" rot="R270">
+<attribute name="OC_NEWARK" value="36M3542" x="11.43" y="44.45" size="1.778" layer="27" rot="R270" display="off"/>
+<attribute name="MPN" value="B3F-1000" x="11.43" y="44.45" size="1.778" layer="27" rot="R270" display="off"/>
+<attribute name="MF" value="" x="11.43" y="44.45" size="1.778" layer="27" rot="R270" display="off"/>
+<attribute name="OC_FARNELL" value="176432" x="11.43" y="44.45" size="1.778" layer="27" rot="R270" display="off"/>
 </element>
-<element name="S2" library="switch-omron" package="B3F-10XX" value="" x="24.13" y="41.91" rot="R90">
-<attribute name="OC_NEWARK" value="36M3542" x="24.13" y="41.91" size="1.778" layer="27" rot="R90" display="off"/>
-<attribute name="MPN" value="B3F-1000" x="24.13" y="41.91" size="1.778" layer="27" rot="R90" display="off"/>
-<attribute name="MF" value="" x="24.13" y="41.91" size="1.778" layer="27" rot="R90" display="off"/>
-<attribute name="OC_FARNELL" value="176432" x="24.13" y="41.91" size="1.778" layer="27" rot="R90" display="off"/>
+<element name="S2" library="switch-omron" package="B3F-10XX" value="" x="22.86" y="44.45" rot="R270">
+<attribute name="OC_NEWARK" value="36M3542" x="22.86" y="44.45" size="1.778" layer="27" rot="R270" display="off"/>
+<attribute name="MPN" value="B3F-1000" x="22.86" y="44.45" size="1.778" layer="27" rot="R270" display="off"/>
+<attribute name="MF" value="" x="22.86" y="44.45" size="1.778" layer="27" rot="R270" display="off"/>
+<attribute name="OC_FARNELL" value="176432" x="22.86" y="44.45" size="1.778" layer="27" rot="R270" display="off"/>
 </element>
-<element name="S3" library="switch-omron" package="B3F-10XX" value="" x="36.83" y="41.91" rot="R270">
-<attribute name="OC_NEWARK" value="36M3542" x="36.83" y="41.91" size="1.778" layer="27" rot="R270" display="off"/>
-<attribute name="MPN" value="B3F-1000" x="36.83" y="41.91" size="1.778" layer="27" rot="R270" display="off"/>
-<attribute name="MF" value="" x="36.83" y="41.91" size="1.778" layer="27" rot="R270" display="off"/>
-<attribute name="OC_FARNELL" value="176432" x="36.83" y="41.91" size="1.778" layer="27" rot="R270" display="off"/>
+<element name="S3" library="switch-omron" package="B3F-10XX" value="" x="34.29" y="44.45" rot="R270">
+<attribute name="OC_NEWARK" value="36M3542" x="34.29" y="44.45" size="1.778" layer="27" rot="R270" display="off"/>
+<attribute name="MPN" value="B3F-1000" x="34.29" y="44.45" size="1.778" layer="27" rot="R270" display="off"/>
+<attribute name="MF" value="" x="34.29" y="44.45" size="1.778" layer="27" rot="R270" display="off"/>
+<attribute name="OC_FARNELL" value="176432" x="34.29" y="44.45" size="1.778" layer="27" rot="R270" display="off"/>
 </element>
-<element name="S4" library="switch-omron" package="B3F-10XX" value="" x="49.53" y="41.91" rot="R270">
-<attribute name="OC_NEWARK" value="36M3542" x="49.53" y="41.91" size="1.778" layer="27" rot="R270" display="off"/>
-<attribute name="MPN" value="B3F-1000" x="49.53" y="41.91" size="1.778" layer="27" rot="R270" display="off"/>
-<attribute name="MF" value="" x="49.53" y="41.91" size="1.778" layer="27" rot="R270" display="off"/>
-<attribute name="OC_FARNELL" value="176432" x="49.53" y="41.91" size="1.778" layer="27" rot="R270" display="off"/>
+<element name="S4" library="switch-omron" package="B3F-10XX" value="" x="45.72" y="44.45" rot="R270">
+<attribute name="OC_NEWARK" value="36M3542" x="45.72" y="44.45" size="1.778" layer="27" rot="R270" display="off"/>
+<attribute name="MPN" value="B3F-1000" x="45.72" y="44.45" size="1.778" layer="27" rot="R270" display="off"/>
+<attribute name="MF" value="" x="45.72" y="44.45" size="1.778" layer="27" rot="R270" display="off"/>
+<attribute name="OC_FARNELL" value="176432" x="45.72" y="44.45" size="1.778" layer="27" rot="R270" display="off"/>
 </element>
 <element name="U$1" library="ESP12E_DEVKIT" package="ESP12E_DEVKIT" value="ESP12E_DEVKIT" x="68.58" y="26.67" rot="R180"/>
-<element name="R1" library="rcl" package="0207/5V" value="4.7K" x="44.45" y="31.75"/>
-<element name="R2" library="rcl" package="0207/5V" value="4.7K" x="44.45" y="25.4"/>
-<element name="R3" library="rcl" package="0207/5V" value="4.7K" x="44.45" y="20.32"/>
-<element name="R4" library="rcl" package="0207/5V" value="4.7K" x="44.45" y="15.24"/>
-<element name="R5" library="rcl" package="0207/5V" value="4.7K" x="44.45" y="10.16"/>
-<element name="R6" library="rcl" package="0207/5V" value="4.7K" x="44.45" y="5.08"/>
+<element name="H1" library="holes" package="3,2" value="MOUNT-HOLE3.2" x="160.02" y="43.18" rot="R90"/>
+<element name="JP1" library="pinhead" package="1X04" value="OLED" x="26.67" y="31.75"/>
 </elements>
 <signals>

Commit message: images and brd update
Parts:
- removed H1: MOUNT-HOLE3.2, holes:3,2
Changed lines of the file:
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@@
 <setting verticaltext="up"/>
 </settings>
-<grid distance="0.05" unitdist="inch" unit="inch" style="lines" multiple="1" display="no" altdistance="0.025" altunitdist="inch" altunit="inch"/>
+<grid distance="7.5" unitdist="mm" unit="mm" style="lines" multiple="1" display="yes" altdistance="0.025" altunitdist="inch" altunit="inch"/>
 <layers>
 <layer number="1" name="Top" color="4" fill="1" visible="yes" active="yes"/>
@@
 <layer number="43" name="vRestrict" color="2" fill="10" visible="yes" active="yes"/>
 <layer number="44" name="Drills" color="7" fill="1" visible="no" active="yes"/>
-<layer number="45" name="Holes" color="7" fill="1" visible="no" active="yes"/>
+<layer number="45" name="Holes" color="7" fill="1" visible="yes" active="yes"/>
 <layer number="46" name="Milling" color="3" fill="1" visible="no" active="yes"/>
 <layer number="47" name="Measures" color="7" fill="1" visible="no" active="yes"/>
@@
 <wire x1="59.36465" y1="0.33181875" x2="53.746" y2="0.216140625" width="0.001" layer="20"/>
 <wire x1="53.746" y1="0.216140625" x2="48.11515" y2="0.14091875" width="0.001" layer="20"/>
+<hole x="163.83" y="43.18" drill="3.2"/>
 </plain>
 <attributes>
@@
 </element>
 <element name="U$1" library="ESP12E_DEVKIT" package="ESP12E_DEVKIT" value="ESP12E_DEVKIT" x="68.58" y="26.67" rot="R180"/>
-<element name="H1" library="holes" package="3,2" value="MOUNT-HOLE3.2" x="160.02" y="43.18" rot="R90"/>
 <element name="JP1" library="pinhead" package="1X04" value="OLED" x="26.67" y="31.75"/>
 </elements>
 <signals>
+<signal name="N$1">
+<via x="12.58" y="19.05" extent="1-16" drill="1.6" shape="square"/>
+<via x="87.58" y="19.05" extent="1-16" drill="1.6" shape="square"/>
+</signal>
 </signals>
 </board>

Commit message: revise component placement in eagle
Parts:
- moved JP1 64.6 mm to (91.0, 37.8), turned to 90 degrees
- moved S4 42.3 mm to (68.3, 8.70)
- moved U$1 42.1 mm to (27.5, 35.8), turned to 270 degrees
- moved S3 41.7 mm to (55.7, 8.70)
- moved S2 41.6 mm to (44.2, 8.70)
- moved S1 41.0 mm to (31.6, 8.70)
Changed lines of the file:
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@@
 <setting verticaltext="up"/>
 </settings>
-<grid distance="7.5" unitdist="mm" unit="mm" style="lines" multiple="1" display="yes" altdistance="0.025" altunitdist="inch" altunit="inch"/>
+<grid distance="1" unitdist="mm" unit="mm" style="lines" multiple="1" display="yes" altdistance="0.025" altunitdist="inch" altunit="inch"/>
 <layers>
 <layer number="1" name="Top" color="4" fill="1" visible="yes" active="yes"/>
@@
 </autorouter>
 <elements>
-<element name="S1" library="switch-omron" package="B3F-10XX" value="" x="11.43" y="44.45" rot="R270">
-<attribute name="OC_NEWARK" value="36M3542" x="11.43" y="44.45" size="1.778" layer="27" rot="R270" display="off"/>
-<attribute name="MPN" value="B3F-1000" x="11.43" y="44.45" size="1.778" layer="27" rot="R270" display="off"/>
-<attribute name="MF" value="" x="11.43" y="44.45" size="1.778" layer="27" rot="R270" display="off"/>
-<attribute name="OC_FARNELL" value="176432" x="11.43" y="44.45" size="1.778" layer="27" rot="R270" display="off"/>
+<element name="S1" library="switch-omron" package="B3F-10XX" value="" x="31.58" y="8.7" rot="R270">
+<attribute name="OC_NEWARK" value="36M3542" x="31.58" y="8.7" size="1.778" layer="27" rot="R270" display="off"/>
+<attribute name="MPN" value="B3F-1000" x="31.58" y="8.7" size="1.778" layer="27" rot="R270" display="off"/>
+<attribute name="MF" value="" x="31.58" y="8.7" size="1.778" layer="27" rot="R270" display="off"/>
+<attribute name="OC_FARNELL" value="176432" x="31.58" y="8.7" size="1.778" layer="27" rot="R270" display="off"/>
 </element>
-<element name="S2" library="switch-omron" package="B3F-10XX" value="" x="22.86" y="44.45" rot="R270">
-<attribute name="OC_NEWARK" value="36M3542" x="22.86" y="44.45" size="1.778" layer="27" rot="R270" display="off"/>
-<attribute name="MPN" value="B3F-1000" x="22.86" y="44.45" size="1.778" layer="27" rot="R270" display="off"/>
-<attribute name="MF" value="" x="22.86" y="44.45" size="1.778" layer="27" rot="R270" display="off"/>
-<attribute name="OC_FARNELL" value="176432" x="22.86" y="44.45" size="1.778" layer="27" rot="R270" display="off"/>
+<element name="S2" library="switch-omron" package="B3F-10XX" value="" x="44.16" y="8.7" rot="R270">
+<attribute name="OC_NEWARK" value="36M3542" x="44.16" y="8.7" size="1.778" layer="27" rot="R270" display="off"/>
+<attribute name="MPN" value="B3F-1000" x="44.16" y="8.7" size="1.778" layer="27" rot="R270" display="off"/>
+<attribute name="MF" value="" x="44.16" y="8.7" size="1.778" layer="27" rot="R270" display="off"/>
+<attribute name="OC_FARNELL" value="176432" x="44.16" y="8.7" size="1.778" layer="27" rot="R270" display="off"/>
 </element>
-<element name="S3" library="switch-omron" package="B3F-10XX" value="" x="34.29" y="44.45" rot="R270">
-<attribute name="OC_NEWARK" value="36M3542" x="34.29" y="44.45" size="1.778" layer="27" rot="R270" display="off"/>
-<attribute name="MPN" value="B3F-1000" x="34.29" y="44.45" size="1.778" layer="27" rot="R270" display="off"/>
-<attribute name="MF" value="" x="34.29" y="44.45" size="1.778" layer="27" rot="R270" display="off"/>
-<attribute name="OC_FARNELL" value="176432" x="34.29" y="44.45" size="1.778" layer="27" rot="R270" display="off"/>
+<element name="S3" library="switch-omron" package="B3F-10XX" value="" x="55.74" y="8.7" rot="R270">
+<attribute name="OC_NEWARK" value="36M3542" x="55.74" y="8.7" size="1.778" layer="27" rot="R270" display="off"/>
+<attribute name="MPN" value="B3F-1000" x="55.74" y="8.7" size="1.778" layer="27" rot="R270" display="off"/>
+<attribute name="MF" value="" x="55.74" y="8.7" size="1.778" layer="27" rot="R270" display="off"/>
+<attribute name="OC_FARNELL" value="176432" x="55.74" y="8.7" size="1.778" layer="27" rot="R270" display="off"/>
 </element>
-<element name="S4" library="switch-omron" package="B3F-10XX" value="" x="45.72" y="44.45" rot="R270">
-<attribute name="OC_NEWARK" value="36M3542" x="45.72" y="44.45" size="1.778" layer="27" rot="R270" display="off"/>
-<attribute name="MPN" value="B3F-1000" x="45.72" y="44.45" size="1.778" layer="27" rot="R270" display="off"/>
-<attribute name="MF" value="" x="45.72" y="44.45" size="1.778" layer="27" rot="R270" display="off"/>
-<attribute name="OC_FARNELL" value="176432" x="45.72" y="44.45" size="1.778" layer="27" rot="R270" display="off"/>
+<element name="S4" library="switch-omron" package="B3F-10XX" value="" x="68.32" y="8.7" rot="R270">
+<attribute name="OC_NEWARK" value="36M3542" x="68.32" y="8.7" size="1.778" layer="27" rot="R270" display="off"/>
+<attribute name="MPN" value="B3F-1000" x="68.32" y="8.7" size="1.778" layer="27" rot="R270" display="off"/>
+<attribute name="MF" value="" x="68.32" y="8.7" size="1.778" layer="27" rot="R270" display="off"/>
+<attribute name="OC_FARNELL" value="176432" x="68.32" y="8.7" size="1.778" layer="27" rot="R270" display="off"/>
 </element>
-<element name="U$1" library="ESP12E_DEVKIT" package="ESP12E_DEVKIT" value="ESP12E_DEVKIT" x="68.58" y="26.67" rot="R180"/>
-<element name="JP1" library="pinhead" package="1X04" value="OLED" x="26.67" y="31.75"/>
+<element name="U$1" library="ESP12E_DEVKIT" package="ESP12E_DEVKIT" value="ESP12E_DEVKIT" x="27.53" y="35.83" rot="R270"/>
+<element name="JP1" library="pinhead" package="1X04" value="OLED" x="91.02" y="37.75" rot="R90"/>
 </elements>
 <signals>
-<signal name="N$1">
-<via x="12.58" y="19.05" extent="1-16" drill="1.6" shape="square"/>
-<via x="87.58" y="19.05" extent="1-16" drill="1.6" shape="square"/>
+<signal name="N$2">
+<via x="19.4" y="19.05" extent="1-16" drill="1.6" shape="square"/>
+<via x="90.9" y="19.05" extent="1-16" drill="1.6" shape="square"/>
 </signal>
 </signals>
