File: eagle/hh.sch (EAGLE design)
At the start: 3 parts

Commit message: updates to eagle files
Parts:
- removed ESP8266(L), ESP8266(R): (no value), pinhead:PINHD-1X15
- removed OLED: (no value), pinhead:PINHD-1X4
- added R1, R2, R3, R4, R5, R6: 4.7K, rcl:R-US_0207/5V
- added S1, S2, S3, S4: (no value), switch-omron:10-XX
- added U$1: ESP12E_DEVKIT, ESP12E_DEVKIT:ESP12E_DEVKIT
Other:
- note removed: "sda scl vcc gnd"
Changed lines of the file:
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@@
 <setting verticaltext="up"/>
 </settings>
-<grid distance="0.1" unitdist="inch" unit="inch" style="lines" multiple="1" display="no" altdistance="0.01" altunitdist="inch" altunit="inch"/>
+<grid distance="0.5" unitdist="inch" unit="inch" style="lines" multiple="1" display="yes" altdistance="0.01" altunitdist="inch" altunit="inch"/>
 <layers>
-<layer number="1" name="Top" color="4" fill="1" visible="yes" active="no"/>
-<layer number="16" name="Bottom" color="1" fill="1" visible="yes" active="no"/>
-<layer number="17" name="Pads" color="2" fill="1" visible="yes" active="no"/>
-<layer number="18" name="Vias" color="2" fill="1" visible="yes" active="no"/>
-<layer number="19" name="Unrouted" color="6" fill="1" visible="yes" active="no"/>
-<layer number="20" name="Dimension" color="15" fill="1" visible="yes" active="no"/>
-<layer number="21" name="tPlace" color="7" fill="1" visible="yes" active="no"/>
-<layer number="22" name="bPlace" color="7" fill="1" visible="yes" active="no"/>
-<layer number="23" name="tOrigins" color="15" fill="1" visible="yes" active="no"/>
-<layer number="24" name="bOrigins" color="15" fill="1" visible="yes" active="no"/>
-<layer number="25" name="tNames" color="7" fill="1" visible="yes" active="no"/>
-<layer number="26" name="bNames" color="7" fill="1" visible="yes" active="no"/>
-<layer number="27" name="tValues" color="7" fill="1" visible="yes" active="no"/>
-<layer number="28" name="bValues" color="7" fill="1" visible="yes" active="no"/>
+<layer number="1" name="Top" color="4" fill="1" visible="no" active="no"/>
+<layer number="16" name="Bottom" color="1" fill="1" visible="no" active="no"/>
+<layer number="17" name="Pads" color="2" fill="1" visible="no" active="no"/>
+<layer number="18" name="Vias" color="2" fill="1" visible="no" active="no"/>
+<layer number="19" name="Unrouted" color="6" fill="1" visible="no" active="no"/>
+<layer number="20" name="Dimension" color="15" fill="1" visible="no" active="no"/>
+<layer number="21" name="tPlace" color="7" fill="1" visible="no" active="no"/>
+<layer number="22" name="bPlace" color="7" fill="1" visible="no" active="no"/>
+<layer number="23" name="tOrigins" color="15" fill="1" visible="no" active="no"/>
+<layer number="24" name="bOrigins" color="15" fill="1" visible="no" active="no"/>
+<layer number="25" name="tNames" color="7" fill="1" visible="no" active="no"/>
+<layer number="26" name="bNames" color="7" fill="1" visible="no" active="no"/>
+<layer number="27" name="tValues" color="7" fill="1" visible="no" active="no"/>
+<layer number="28" name="bValues" color="7" fill="1" visible="no" active="no"/>
 <layer number="29" name="tStop" color="7" fill="3" visible="no" active="no"/>
 <layer number="30" name="bStop" color="7" fill="6" visible="no" active="no"/>
@@
 <layer number="35" name="tGlue" color="7" fill="4" visible="no" active="no"/>
 <layer number="36" name="bGlue" color="7" fill="5" visible="no" active="no"/>
-<layer number="37" name="tTest" color="7" fill="1" visible="yes" active="no"/>
-<layer number="38" name="bTest" color="7" fill="1" visible="yes" active="no"/>
+<layer number="37" name="tTest" color="7" fill="1" visible="no" active="no"/>
+<layer number="38" name="bTest" color="7" fill="1" visible="no" active="no"/>
 <layer number="39" name="tKeepout" color="4" fill="11" visible="no" active="no"/>
 <layer number="40" name="bKeepout" color="1" fill="11" visible="no" active="no"/>
@@
 <layer number="44" name="Drills" color="7" fill="1" visible="no" active="no"/>
 <layer number="45" name="Holes" color="7" fill="1" visible="no" active="no"/>
-<layer number="46" name="Milling" color="3" fill="1" visible="yes" active="no"/>
-<layer number="47" name="Measures" color="7" fill="1" visible="yes" active="no"/>
-<layer number="48" name="Document" color="7" fill="1" visible="yes" active="no"/>
-<layer number="49" name="Reference" color="7" fill="1" visible="yes" active="no"/>
-<layer number="51" name="tDocu" color="7" fill="1" visible="yes" active="no"/>
-<layer number="52" name="bDocu" color="7" fill="1" visible="yes" active="no"/>
+<layer number="46" name="Milling" color="3" fill="1" visible="no" active="no"/>
+<layer number="47" name="Measures" color="7" fill="1" visible="no" active="no"/>
+<layer number="48" name="Document" color="7" fill="1" visible="no" active="no"/>
+<layer number="49" name="Reference" color="7" fill="1" visible="no" active="no"/>
+<layer number="51" name="tDocu" color="7" fill="1" visible="no" active="no"/>
+<layer number="52" name="bDocu" color="7" fill="1" visible="no" active="no"/>
 <layer number="90" name="Modules" color="5" fill="1" visible="yes" active="yes"/>
 <layer number="91" name="Nets" color="2" fill="1" visible="yes" active="yes"/>
@@
 </classes>
 <parts>
-<part name="ESP8266(L)" library="pinhead" deviceset="PINHD-1X15" device=""/>
-<part name="ESP8266(R)" library="pinhead" deviceset="PINHD-1X15" device=""/>
-<part name="OLED" library="pinhead" deviceset="PINHD-1X4" device=""/>
+<part name="S1" library="switch-omron" deviceset="10-XX" device=""/>
+<part name="S2" library="switch-omron" deviceset="10-XX" device=""/>
+<part name="S3" library="switch-omron" deviceset="10-XX" device=""/>
+<part name="S4" library="switch-omron" deviceset="10-XX" device=""/>
+<part name="U$1" library="ESP12E_DEVKIT" deviceset="ESP12E_DEVKIT" device=""/>
+<part name="R1" library="rcl" deviceset="R-US_" device="0207/5V" value="4.7K"/>
+<part name="R2" library="rcl" deviceset="R-US_" device="0207/5V" value="4.7K"/>
+<part name="R3" library="rcl" deviceset="R-US_" device="0207/5V" value="4.7K"/>
+<part name="R4" library="rcl" deviceset="R-US_" device="0207/5V" value="4.7K"/>
+<part name="R5" library="rcl" deviceset="R-US_" device="0207/5V" value="4.7K"/>
+<part name="R6" library="rcl" deviceset="R-US_" device="0207/5V" value="4.7K"/>
+<part name="FRAME1" library="frames" deviceset="FRAME_A_L" device=""/>
+<part name="GND1" library="supply1" deviceset="GND" device=""/>
+<part name="GND2" library="supply1" deviceset="GND" device=""/>
+<part name="P+1" library="supply1" deviceset="VCC" device=""/>
+<part name="P+2" library="supply1" deviceset="VCC" device=""/>
 </parts>
 <sheets>
@@
 <description>hackharder</description>
 <plain>
-<text x="20.32" y="96.52" size="1.778" layer="91">sda
-scl
-vcc
-gnd</text>
 </plain>
 <instances>
-<instance part="ESP8266(L)" gate="A" x="35.56" y="53.34"/>
-<instance part="ESP8266(R)" gate="A" x="63.5" y="53.34"/>
-<instance part="OLED" gate="A" x="33.02" y="99.06"/>
+<instance part="S1" gate="1" x="22.86" y="142.24"/>
+<instance part="S2" gate="1" x="22.86" y="119.38"/>
+<instance part="S3" gate="1" x="22.86" y="91.44"/>
+<instance part="S4" gate="1" x="22.86" y="68.58"/>
+<instance part="U$1" gate="G$1" x="119.38" y="93.98"/>
+<instance part="R1" gate="G$1" x="147.32" y="162.56"/>
+<instance part="R2" gate="G$1" x="147.32" y="139.7"/>
+<instance part="R3" gate="G$1" x="58.42" y="147.32"/>
+<instance part="R4" gate="G$1" x="58.42" y="121.92"/>
+<instance part="R5" gate="G$1" x="55.88" y="93.98"/>
+<instance part="R6" gate="G$1" x="53.34" y="63.5"/>
+<instance part="FRAME1" gate="G$1" x="-22.86" y="-12.7"/>
+<instance part="FRAME1" gate="G$2" x="149.86" y="-12.7"/>
+<instance part="GND1" gate="1" x="88.9" y="50.8"/>
+<instance part="GND2" gate="1" x="38.1" y="50.8"/>
+<instance part="P+1" gate="VCC" x="76.2" y="50.8" rot="R90"/>
+<instance part="P+2" gate="VCC" x="76.2" y="50.8" rot="R90"/>
 </instances>
 <busses>
 </busses>
 <nets>
+<net name="VCC" class="0">
+<segment>
+<pinref part="P+1" gate="VCC" pin="VCC"/>
+<pinref part="P+2" gate="VCC" pin="VCC"/>
+</segment>
+</net>
 </nets>
 </sheet>
@@
 </schematic>
 </drawing>
-<compatibility>
-<note version="6.3" minversion="6.2.2" severity="warning">
-Since Version 6.2.2 text objects can contain more than one line,
-which will not be processed correctly with this version.
-</note>
-</compatibility>
 </eagle>

Commit message: design updates
Parts:
- removed R1, R2, R3, R4, R5, R6: 4.7K, rcl:R-US_0207/5V
- added H1: MOUNT-HOLE3.2, holes:MOUNT-HOLE3.2
- added JP1: OLED, pinhead:PINHD-1X4
Changed lines of the file:
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@@
 <part name="S4" library="switch-omron" deviceset="10-XX" device=""/>
 <part name="U$1" library="ESP12E_DEVKIT" deviceset="ESP12E_DEVKIT" device=""/>
-<part name="R1" library="rcl" deviceset="R-US_" device="0207/5V" value="4.7K"/>
-<part name="R2" library="rcl" deviceset="R-US_" device="0207/5V" value="4.7K"/>
-<part name="R3" library="rcl" deviceset="R-US_" device="0207/5V" value="4.7K"/>
-<part name="R4" library="rcl" deviceset="R-US_" device="0207/5V" value="4.7K"/>
-<part name="R5" library="rcl" deviceset="R-US_" device="0207/5V" value="4.7K"/>
-<part name="R6" library="rcl" deviceset="R-US_" device="0207/5V" value="4.7K"/>
 <part name="FRAME1" library="frames" deviceset="FRAME_A_L" device=""/>
 <part name="GND1" library="supply1" deviceset="GND" device=""/>
@@
 <part name="P+1" library="supply1" deviceset="VCC" device=""/>
 <part name="P+2" library="supply1" deviceset="VCC" device=""/>
+<part name="H1" library="holes" deviceset="MOUNT-HOLE" device="3.2"/>
+<part name="JP1" library="pinhead" deviceset="PINHD-1X4" device="" value="OLED"/>
 </parts>
 <sheets>
@@
 <instance part="S4" gate="1" x="22.86" y="68.58"/>
 <instance part="U$1" gate="G$1" x="119.38" y="93.98"/>
-<instance part="R1" gate="G$1" x="147.32" y="162.56"/>
-<instance part="R2" gate="G$1" x="147.32" y="139.7"/>
-<instance part="R3" gate="G$1" x="58.42" y="147.32"/>
-<instance part="R4" gate="G$1" x="58.42" y="121.92"/>
-<instance part="R5" gate="G$1" x="55.88" y="93.98"/>
-<instance part="R6" gate="G$1" x="53.34" y="63.5"/>
 <instance part="FRAME1" gate="G$1" x="-22.86" y="-12.7"/>
 <instance part="FRAME1" gate="G$2" x="149.86" y="-12.7"/>
@@
 <instance part="P+1" gate="VCC" x="76.2" y="50.8" rot="R90"/>
 <instance part="P+2" gate="VCC" x="76.2" y="50.8" rot="R90"/>
+<instance part="H1" gate="G$1" x="12.7" y="177.8"/>
+<instance part="JP1" gate="A" x="76.2" y="165.1"/>
 </instances>
 <busses>

Commit message: images and brd update
Parts:
- removed H1: MOUNT-HOLE3.2, holes:MOUNT-HOLE3.2
Changed lines of the file:
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@@
 <part name="P+1" library="supply1" deviceset="VCC" device=""/>
 <part name="P+2" library="supply1" deviceset="VCC" device=""/>
-<part name="H1" library="holes" deviceset="MOUNT-HOLE" device="3.2"/>
 <part name="JP1" library="pinhead" deviceset="PINHD-1X4" device="" value="OLED"/>
 </parts>
@@
 <instance part="P+1" gate="VCC" x="76.2" y="50.8" rot="R90"/>
 <instance part="P+2" gate="VCC" x="76.2" y="50.8" rot="R90"/>
-<instance part="H1" gate="G$1" x="12.7" y="177.8"/>
 <instance part="JP1" gate="A" x="76.2" y="165.1"/>
 </instances>

Commit message: wiring 1
Connections:
- new net GND: U$1.GND@3
- new net N$1: U$1.3V3@2
- new net N$3: JP1.1, U$1.3V3@1
- new net N$4: JP1.2, U$1.GND@2
- new net N$5: JP1.3, U$1.D1
- new net N$6: JP1.4, U$1.D2
Other:
- moved on the sheet: JP1, U$1
Changed lines of the file:
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@@
 <setting verticaltext="up"/>
 </settings>
-<grid distance="0.5" unitdist="inch" unit="inch" style="lines" multiple="1" display="yes" altdistance="0.01" altunitdist="inch" altunit="inch"/>
+<grid distance="0.1" unitdist="inch" unit="inch" style="lines" multiple="1" display="no" altdistance="0.01" altunitdist="inch" altunit="inch"/>
 <layers>
 <layer number="1" name="Top" color="4" fill="1" visible="no" active="no"/>
@@
 <part name="U$1" library="ESP12E_DEVKIT" deviceset="ESP12E_DEVKIT" device=""/>
 <part name="FRAME1" library="frames" deviceset="FRAME_A_L" device=""/>
-<part name="GND1" library="supply1" deviceset="GND" device=""/>
 <part name="GND2" library="supply1" deviceset="GND" device=""/>
-<part name="P+1" library="supply1" deviceset="VCC" device=""/>
 <part name="P+2" library="supply1" deviceset="VCC" device=""/>
 <part name="JP1" library="pinhead" deviceset="PINHD-1X4" device="" value="OLED"/>
@@
 <instance part="S3" gate="1" x="22.86" y="91.44"/>
 <instance part="S4" gate="1" x="22.86" y="68.58"/>
-<instance part="U$1" gate="G$1" x="119.38" y="93.98"/>
+<instance part="U$1" gate="G$1" x="119.38" y="93.98" rot="R180"/>
 <instance part="FRAME1" gate="G$1" x="-22.86" y="-12.7"/>
 <instance part="FRAME1" gate="G$2" x="149.86" y="-12.7"/>
-<instance part="GND1" gate="1" x="88.9" y="50.8"/>
-<instance part="GND2" gate="1" x="38.1" y="50.8"/>
-<instance part="P+1" gate="VCC" x="76.2" y="50.8" rot="R90"/>
-<instance part="P+2" gate="VCC" x="76.2" y="50.8" rot="R90"/>
-<instance part="JP1" gate="A" x="76.2" y="165.1"/>
+<instance part="GND2" gate="1" x="78.74" y="129.54"/>
+<instance part="P+2" gate="VCC" x="88.9" y="129.54" rot="R90"/>
+<instance part="JP1" gate="A" x="81.28" y="45.72" rot="R90"/>
 </instances>
 <busses>
 </busses>
 <nets>
-<net name="VCC" class="0">
+<net name="GND" class="0">
 <segment>
-<pinref part="P+1" gate="VCC" pin="VCC"/>
-<pinref part="P+2" gate="VCC" pin="VCC"/>
+<pinref part="U$1" gate="G$1" pin="GND@3"/>
+<pinref part="GND2" gate="1" pin="GND"/>
+<wire x1="101.6" y1="109.22" x2="78.74" y2="109.22" width="0.1524" layer="91"/>
+<wire x1="78.74" y1="109.22" x2="78.74" y2="132.08" width="0.1524" layer="91"/>
 </segment>
 </net>
+<net name="N$1" class="0">
+<segment>
+<pinref part="U$1" gate="G$1" pin="3V3@2"/>
+<wire x1="88.9" y1="129.54" x2="88.9" y2="124.46" width="0.1524" layer="91"/>
+<wire x1="88.9" y1="124.46" x2="101.6" y2="111.76" width="0.1524" layer="91"/>
+</segment>
+</net>
+<net name="N$3" class="0">
+<segment>
+<pinref part="JP1" gate="A" pin="1"/>
+<pinref part="U$1" gate="G$1" pin="3V3@1"/>
+<wire x1="76.2" y1="43.18" x2="76.2" y2="63.5" width="0.1524" layer="91"/>
+<wire x1="76.2" y1="63.5" x2="101.6" y2="88.9" width="0.1524" layer="91"/>
+</segment>
+</net>
+<net name="N$4" class="0">
+<segment>
+<pinref part="JP1" gate="A" pin="2"/>
+<pinref part="U$1" gate="G$1" pin="GND@2"/>
+<wire x1="78.74" y1="43.18" x2="78.74" y2="68.58" width="0.1524" layer="91"/>
+<wire x1="78.74" y1="68.58" x2="101.6" y2="91.44" width="0.1524" layer="91"/>
+</segment>
+</net>
+<net name="N$6" class="0">
+<segment>
+<pinref part="JP1" gate="A" pin="4"/>
+<pinref part="U$1" gate="G$1" pin="D2"/>
+<wire x1="83.82" y1="43.18" x2="83.82" y2="63.5" width="0.1524" layer="91"/>
+<wire x1="83.82" y1="63.5" x2="101.6" y2="81.28" width="0.1524" layer="91"/>
+</segment>
+</net>
+<net name="N$5" class="0">
+<segment>
+<pinref part="JP1" gate="A" pin="3"/>
+<pinref part="U$1" gate="G$1" pin="D1"/>
+<wire x1="81.28" y1="43.18" x2="81.28" y2="58.42" width="0.1524" layer="91"/>
+<wire x1="81.28" y1="58.42" x2="101.6" y2="78.74" width="0.1524" layer="91"/>
+</segment>
+</net>

Commit message: wiring 2
Connections:
- new net N$2: S4.S, S4.S1, U$1.D3
- new net N$7: S3.S, S3.S1, U$1.D4
- new net N$8: S2.S, S2.S1, U$1.D5
- new net N$9: S1.S, S1.S1, U$1.D6
- net GND: now also S1.P, S1.P1, S2.P, S2.P1, S3.P, S3.P1, S4.P, S4.P1
Changed lines of the file:
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@@
 <pinref part="GND2" gate="1" pin="GND"/>
 <wire x1="101.6" y1="109.22" x2="78.74" y2="109.22" width="0.1524" layer="91"/>
-<wire x1="78.74" y1="109.22" x2="78.74" y2="132.08" width="0.1524" layer="91"/>
+<wire x1="78.74" y1="109.22" x2="78.74" y2="129.54" width="0.1524" layer="91"/>
+<pinref part="S4" gate="1" pin="P"/>
+<wire x1="78.74" y1="129.54" x2="78.74" y2="132.08" width="0.1524" layer="91"/>
+<wire x1="22.86" y1="63.5" x2="10.16" y2="63.5" width="0.1524" layer="91"/>
+<wire x1="10.16" y1="63.5" x2="10.16" y2="86.36" width="0.1524" layer="91"/>
+<wire x1="10.16" y1="86.36" x2="10.16" y2="114.3" width="0.1524" layer="91"/>
+<wire x1="10.16" y1="114.3" x2="10.16" y2="137.16" width="0.1524" layer="91"/>
+<wire x1="10.16" y1="137.16" x2="10.16" y2="157.48" width="0.1524" layer="91"/>
+<wire x1="10.16" y1="157.48" x2="71.12" y2="157.48" width="0.1524" layer="91"/>
+<wire x1="71.12" y1="157.48" x2="71.12" y2="129.54" width="0.1524" layer="91"/>
+<wire x1="71.12" y1="129.54" x2="78.74" y2="129.54" width="0.1524" layer="91"/>
+<junction x="78.74" y="129.54"/>
+<pinref part="S3" gate="1" pin="P"/>
+<wire x1="22.86" y1="86.36" x2="10.16" y2="86.36" width="0.1524" layer="91"/>
+<junction x="10.16" y="86.36"/>
+<pinref part="S2" gate="1" pin="P"/>
+<wire x1="22.86" y1="114.3" x2="10.16" y2="114.3" width="0.1524" layer="91"/>
+<junction x="10.16" y="114.3"/>
+<pinref part="S1" gate="1" pin="P"/>
+<wire x1="22.86" y1="137.16" x2="10.16" y2="137.16" width="0.1524" layer="91"/>
+<junction x="10.16" y="137.16"/>
+<pinref part="S1" gate="1" pin="P1"/>
+<wire x1="25.4" y1="137.16" x2="22.86" y2="137.16" width="0.1524" layer="91"/>
+<junction x="22.86" y="137.16"/>
+<pinref part="S2" gate="1" pin="P1"/>
+<wire x1="25.4" y1="114.3" x2="22.86" y2="114.3" width="0.1524" layer="91"/>
+<junction x="22.86" y="114.3"/>
+<pinref part="S3" gate="1" pin="P1"/>
+<wire x1="25.4" y1="86.36" x2="22.86" y2="86.36" width="0.1524" layer="91"/>
+<junction x="22.86" y="86.36"/>
+<pinref part="S4" gate="1" pin="P1"/>
+<wire x1="25.4" y1="63.5" x2="22.86" y2="63.5" width="0.1524" layer="91"/>
+<junction x="22.86" y="63.5"/>
 </segment>
 </net>
@@
 </segment>
 </net>
+<net name="N$2" class="0">
+<segment>
+<pinref part="U$1" gate="G$1" pin="D3"/>
+<pinref part="S4" gate="1" pin="S1"/>
+<wire x1="101.6" y1="83.82" x2="35.56" y2="83.82" width="0.1524" layer="91"/>
+<wire x1="35.56" y1="83.82" x2="25.4" y2="73.66" width="0.1524" layer="91"/>
+<pinref part="S4" gate="1" pin="S"/>
+<wire x1="22.86" y1="73.66" x2="25.4" y2="73.66" width="0.1524" layer="91"/>
+<junction x="25.4" y="73.66"/>
+</segment>
+</net>
+<net name="N$7" class="0">
+<segment>
+<pinref part="U$1" gate="G$1" pin="D4"/>
+<pinref part="S3" gate="1" pin="S1"/>
+<wire x1="101.6" y1="86.36" x2="35.56" y2="86.36" width="0.1524" layer="91"/>
+<wire x1="35.56" y1="86.36" x2="25.4" y2="96.52" width="0.1524" layer="91"/>
+<pinref part="S3" gate="1" pin="S"/>
+<wire x1="22.86" y1="96.52" x2="25.4" y2="96.52" width="0.1524" layer="91"/>
+<junction x="25.4" y="96.52"/>
+</segment>
+</net>
+<net name="N$8" class="0">
+<segment>
+<pinref part="U$1" gate="G$1" pin="D5"/>
+<pinref part="S2" gate="1" pin="S1"/>
+<wire x1="101.6" y1="93.98" x2="55.88" y2="93.98" width="0.1524" layer="91"/>
+<wire x1="55.88" y1="93.98" x2="25.4" y2="124.46" width="0.1524" layer="91"/>
+<pinref part="S2" gate="1" pin="S"/>
+<wire x1="22.86" y1="124.46" x2="25.4" y2="124.46" width="0.1524" layer="91"/>
+<junction x="25.4" y="124.46"/>
+</segment>
+</net>
+<net name="N$9" class="0">
+<segment>
+<pinref part="U$1" gate="G$1" pin="D6"/>
+<pinref part="S1" gate="1" pin="S1"/>
+<wire x1="101.6" y1="96.52" x2="76.2" y2="96.52" width="0.1524" layer="91"/>
+<wire x1="76.2" y1="96.52" x2="25.4" y2="147.32" width="0.1524" layer="91"/>
+<pinref part="S1" gate="1" pin="S"/>
+<wire x1="22.86" y1="147.32" x2="25.4" y2="147.32" width="0.1524" layer="91"/>
+<junction x="25.4" y="147.32"/>
+</segment>
+</net>
